Commit message: Fix right gripper rendering: unit declaration and mirror mesh
- finger.dae: meter="1"→meter="0.001" so mm coordinates render at correct scale
- finger_right.dae/stl: y-mirrored right-finger mesh (x=[0,40], y=[0,25.8])
- panda.urdf: right finger uses finger_right.dae with rpy=0 (no rotation needed)

Co-Authored-By: Claude Sonnet 4.6 <noreply@anthropic.com>

File: results/robot_models/panda.urdf (robot description, URDF)
Before this commit: robot panda, 12 links, 11 joints
Links:
- link panda_rightfinger: geometry collision mesh filename=franka_description/meshes/collision/finger.stl; visual mesh filename=franka_description/meshes/visual/finger_right.dae

Commit message: Soft finger: correct frame (outward +Z), black UMI material
Root cause: the soft-gripper STL was authored in a different frame than the
Franka finger link — it extends -Z (into the hand) and is offset in X, so
both fingers pointed inward. Remap into the Franka finger frame:
  X=(x-20)/1000 (center), Y=-y/1000 (body +Y), Z=-z/1000 (extend +Z outward).

- soft_finger.stl: meter-scale, franka-frame binary STL used for both fingers
  (right finger via the stock 180° Z rotation), so they mirror correctly.
- panda.urdf: both finger visuals -> soft_finger.stl + black material (UMI).
- Drop hand-rolled finger_right.dae/stl (replaced by the single framed STL).

Co-Authored-By: Claude Opus 4.8 (1M context) <noreply@anthropic.com>

File: results/robot_models/panda.urdf (robot description, URDF)
Before this commit: robot panda, 12 links, 11 joints
Links:
- link panda_leftfinger: geometry collision mesh filename=franka_description/meshes/collision/finger.stl; visual mesh filename=franka_description/meshes/visual/soft_finger.stl
- link panda_rightfinger: geometry collision mesh filename=franka_description/meshes/collision/finger.stl; visual mesh filename=franka_description/meshes/visual/soft_finger.stl
