Commit message: update model

File: results/robot_models/panda.urdf (robot description, URDF)
Before this commit: robot panda, 12 links, 11 joints
Links:
- link panda_leftfinger: geometry collision mesh filename=franka_description/meshes/collision/finger.stl; visual mesh filename=franka_description/meshes/visual/soft_gripper_finger.stl scale=0.001 0.001 0.001
- link panda_rightfinger: geometry collision mesh filename=franka_description/meshes/collision/finger.stl; visual mesh filename=franka_description/meshes/visual/soft_gripper_finger.stl scale=0.001 0.001 0.001

Commit message: update model

File: results/robot_models/panda.urdf (robot description, URDF)
Before this commit: robot panda, 12 links, 11 joints
Links:
- link panda_leftfinger: geometry collision mesh filename=franka_description/meshes/collision/finger.stl; visual mesh filename=franka_description/meshes/visual/finger.stl scale=0.001 0.001 0.001
- link panda_rightfinger: geometry collision mesh filename=franka_description/meshes/collision/finger.stl; visual mesh filename=franka_description/meshes/visual/finger.stl scale=0.001 0.001 0.001
